File: KSS_V50_HW/MCU.kicad_sch (KiCad schematic)
At the start: 16 parts, among them J4 Conn_01x02_Socket, Q6 SSM3J332R,LF, SW2 SW_SP3T, U10 ATtiny3226-X, U11 AT42QT1010-TSHR

Commit message: Added fab outputs
Parts:
- SW2: DPN (none) -> 563-1035-1-ND; MPN (none) -> CS-4-13NTA
Changed lines of the file:
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@@
+			)
+		)
+		(property "DPN" "563-1035-1-ND"
+			(at 105.41 144.78 0)
+			(effects
+				(font
+					(size 1.27 1.27)
+				)
+				(hide yes)
+			)
+		)
+		(property "MPN" "CS-4-13NTA "
+			(at 105.41 144.78 0)
+			(effects
+				(font
+					(size 1.27 1.27)
+				)
+				(hide yes)
 			)
 		)
