File: KSS_V50_HW/MCU.kicad_sch (KiCad schematic)
At the start: 16 parts, among them J4 Conn_01x02_Socket, Q6 SSM3J332R,LF, SW2 SW_SP3T, U10 ATtiny3226-X, U11 AT42QT1010-TSHR

Commit message: post assembly commit
Parts:
- C30, C31: JLC_PN (none) -> C92490
- C32: JLC_PN (none) -> C113811
- C33: JLC_PN (none) -> C519404
- Q6: JLC_PN (none) -> C146367
- R30, R31, R36, R37: JLC_PN (none) -> C105580
- R33, R34, R35: JLC_PN (none) -> C105578
- SW2: DPN (none) -> 563-1035-1-ND; JLC_PN (none) -> C2921702 Copy; MPN (none) -> CS-4-13NTA
- U10: JLC_PN (none) -> C3235640; MPN (none) -> ATTINY3226-XF
- U11: JLC_PN (none) -> C74512
Changed lines of the file:
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@@
 	(label "SDA"
 		(at 168.91 102.87 0)
-		(fields_autoplaced yes)
 		(effects
 			(font
@@
 	(label "MODE_SW_1"
 		(at 172.72 107.95 180)
-		(fields_autoplaced yes)
 		(effects
 			(font
@@
 	(label "MOT_STBY"
 		(at 187.96 53.34 0)
-		(fields_autoplaced yes)
 		(effects
 			(font
@@
 	(label "SCL"
 		(at 140.97 41.91 180)
-		(fields_autoplaced yes)
 		(effects
 			(font
@@
 	(label "MCU_TX"
 		(at 172.72 80.01 180)
-		(fields_autoplaced yes)
 		(effects
 			(font
@@
 	(label "SDA"
 		(at 160.02 41.91 180)
-		(fields_autoplaced yes)
 		(effects
 			(font
@@
 	(label "MODE_SW_2"
 		(at 87.63 144.78 0)
-		(fields_autoplaced yes)
 		(effects
 			(font
@@
 	(label "MODE_SW_1"
 		(at 87.63 142.24 0)
-		(fields_autoplaced yes)
 		(effects
 			(font
@@
 	(label "CAP_SNS_OUT"
 		(at 152.4 148.59 0)
-		(fields_autoplaced yes)
 		(effects
 			(font
@@
 	(label "MCU_RX"
 		(at 172.72 82.55 180)
-		(fields_autoplaced yes)
 		(effects
 			(font
@@
 	(label "SCL"
 		(at 168.91 100.33 0)
-		(fields_autoplaced yes)
 		(effects
 			(font
@@
 	(label "CAP_SNS_OUT"
 		(at 111.76 105.41 0)
-		(fields_autoplaced yes)
 		(effects
 			(font
@@
 	(label "MOT_STBY"
 		(at 111.76 107.95 0)
-		(fields_autoplaced yes)
 		(effects
 			(font
@@
 	(label "MODE_SW_2"
 		(at 172.72 110.49 180)
-		(fields_autoplaced yes)
 		(effects
 			(font
@@
 		(shape output)
 		(at 109.22 102.87 180)
-		(fields_autoplaced yes)
 		(effects
 			(font
@@
 		(shape output)
 		(at 185.42 95.25 0)
-		(fields_autoplaced yes)
 		(effects
 			(font
@@
 		(shape output)
 		(at 185.42 113.03 0)
-		(fields_autoplaced yes)
 		(effects
 			(font
@@
 		(shape bidirectional)
 		(at 185.42 77.47 0)
-		(fields_autoplaced yes)
 		(effects
 			(font
@@
 		(shape input)
 		(at 185.42 90.17 0)
-		(fields_autoplaced yes)
 		(effects
 			(font
@@
 		(shape output)
 		(at 226.06 38.1 0)
-		(fields_autoplaced yes)
 		(effects
 			(font
@@
 		(shape input)
 		(at 185.42 102.87 0)
-		(fields_autoplaced yes)
 		(effects
 			(font
@@
 		(shape input)
 		(at 185.42 100.33 0)
-		(fields_autoplaced yes)
 		(effects
 			(font
@@
 		(shape input)
 		(at 185.42 82.55 0)
-		(fields_autoplaced yes)
 		(effects
 			(font
@@
 		(shape output)
 		(at 185.42 92.71 0)
-		(fields_autoplaced yes)
 		(effects
 			(font
@@
 		(shape output)
 		(at 185.42 85.09 0)
-		(fields_autoplaced yes)
 		(effects
 			(font
@@
 		(shape output)
 		(at 185.42 80.01 0)
-		(fields_autoplaced yes)
 		(effects
 			(font
@@
 		(shape output)
 		(at 185.42 87.63 0)
-		(fields_autoplaced yes)
 		(effects
 			(font
@@
 		(shape input)
 		(at 109.22 100.33 180)
-		(fields_autoplaced yes)
 		(effects
 			(font
@@
 		(shape output)
 		(at 185.42 105.41 0)
-		(fields_autoplaced yes)
 		(effects
 			(font
@@
 			)
 		)
+		(property "JLC_PN" "C105580"
+			(at 154.94 34.29 0)
+			(effects
+				(font
+					(size 1.27 1.27)
+				)
+				(hide yes)
+			)
+		)
 		(pin "2"
 		)
@@
 			)
 		)
+		(property "JLC_PN" "C105578"
+			(at 73.66 133.35 0)
+			(effects
+				(font
+					(size 1.27 1.27)
+				)
+				(hide yes)
+			)
+		)
 		(pin "2"
 		)
@@
 			)
 		)
+		(property "JLC_PN" ""
+			(at 243.84 143.51 0)
+			(effects
+				(font
+					(size 1.27 1.27)
+				)
+				(hide yes)
+			)
+		)
 		(pin "1"
 		)
@@
 		)
 		(property "DKN" ""
+			(at 179.07 148.59 0)
+			(effects
+				(font
+					(size 1.27 1.27)
+				)
+				(hide yes)
+			)
+		)
+		(property "JLC_PN" "C105580"
 			(at 179.07 148.59 0)
 			(effects
@@
 			)
 		)
+		(property "JLC_PN" "C146367"
+			(at 212.09 40.64 0)
+			(effects
+				(font
+					(size 1.27 1.27)
+				)
+				(hide yes)
+			)
+		)
 		(pin "3"
 		)
@@
 			)
 		)
+		(property "MPN" "ATTINY3226-XF "
+			(at 140.97 95.25 0)
+			(effects
+				(font
+					(size 1.27 1.27)
+				)
+				(hide yes)
+			)
+		)
+		(property "JLC_PN" "C3235640"
+			(at 140.97 95.25 0)
+			(effects
+				(font
+					(size 1.27 1.27)
+				)
+				(hide yes)
+			)
+		)
 		(pin "8"
 		)
@@
 			)
 		)
+		(property "JLC_PN" "C105580"
+			(at 135.89 34.29 0)
+			(effects
+				(font
+					(size 1.27 1.27)
+				)
+				(hide yes)
+			)
+		)
 		(pin "2"
 		)
@@
 			)
 		)
+		(property "JLC_PN" "C519404"
+			(at 170.18 154.94 0)
+			(effects
+				(font
+					(size 1.27 1.27)
+				)
+				(hide yes)
+			)
+		)
 		(pin "2"
 		)
@@
 		)
 		(property "DKN" ""
+			(at 201.93 128.27 0)
+			(effects
+				(font
+					(size 1.27 1.27)
+				)
+				(hide yes)
+			)
+		)
+		(property "JLC_PN" "C92490"
 			(at 201.93 128.27 0)
 			(effects
@@
 			)
 		)
+		(property "MPN" "CS-4-13NTA"
+			(at 105.41 144.78 0)
+			(effects
+				(font
+					(size 1.27 1.27)
+				)
+				(hide yes)
+			)
+		)
+		(property "DPN" "563-1035-1-ND"
+			(at 105.41 144.78 0)
+			(effects
+				(font
+					(size 1.27 1.27)
+				)
+				(hide yes)
+			)
+		)
+		(property "JLC_PN" "C2921702 Copy "
+			(at 105.41 144.78 0)
+			(effects
+				(font
+					(size 1.27 1.27)
+				)
+				(hide yes)
+			)
+		)
 		(pin "4"
 		)
@@
 			)
 		)
+		(property "JLC_PN" "C74512"
+			(at 195.58 146.05 0)
+			(effects
+				(font
+					(size 1.27 1.27)
+				)
+				(hide yes)
+			)
+		)
 		(pin "1"
 		)
@@
 			)
 		)
+		(property "JLC_PN" "C105580"
+			(at 229.87 143.51 0)
+			(effects
+				(font
+					(size 1.27 1.27)
+				)
+				(hide yes)
+			)
+		)
 		(pin "2"
 		)
@@
 		)
 		(property "DKN" ""
+			(at 83.82 133.35 0)
+			(effects
+				(font
+					(size 1.27 1.27)
+				)
+				(hide yes)
+			)
+		)
+		(property "JLC_PN" "C105578"
 			(at 83.82 133.35 0)
 			(effects
@@
 			)
 		)
+		(property "JLC_PN" "C92490"
+			(at 119.38 72.39 0)
+			(effects
+				(font
+					(size 1.27 1.27)
+				)
+				(hide yes)
+			)
+		)
 		(pin "2"
 		)
@@
 			)
 		)
+		(property "JLC_PN" "C113811"
+			(at 215.9 149.86 0)
+			(effects
+				(font
+					(size 1.27 1.27)
+				)
+				(hide yes)
+			)
+		)
 		(pin "2"
 		)
@@
 			(at 204.47 45.72 0)
 			(effects
+				(font
+					(size 1.27 1.27)
+				)
+				(hide yes)
+			)
+		)
+		(property "JLC_PN" "C105578"
+			(at 204.47 45.72 0)
+			(effects
