File: KSS_V50_HW/2_5V_Buck_Boost.kicad_sch (KiCad schematic)
At the start: 10 parts, among them U5 TPS62843

Commit message: post assembly commit
Parts:
- C16, C17, C28, C29: DPN 490-GRM21BZ71E106KE15LCT-ND -> 490-6473-1-ND; Dialectric X7R -> X5R; JLC_PN (none) -> C237493; MPN GRM21BZ71E106KE15L -> GRM21BR61C106KE15K; Voltage Rating 25V -> 16V
- L2: footprint Inductor_SMD:L_Murata_DFE201610P -> ap_built:L_Murata_DFE201610P; JLC_PN (none) -> C882953
- R17: JLC_PN (none) -> C95684
- R32: JLC_PN (none) -> C114626
- U5: JLC_PN (none) -> C25838674
Changed lines of the file:
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@@
 		(shape input)
 		(at 62.23 88.9 180)
-		(fields_autoplaced yes)
 		(effects
 			(font
@@
 			)
 		)
-		(property "MPN" "GRM21BZ71E106KE15L"
+		(property "MPN" "GRM21BR61C106KE15K"
 			(at 224.79 111.76 0)
 			(effects
@@
 			)
 		)
-		(property "DPN" "490-GRM21BZ71E106KE15LCT-ND"
+		(property "DPN" "490-6473-1-ND"
 			(at 224.79 111.76 0)
 			(effects
@@
 			)
 		)
-		(property "Dialectric" "X7R"
+		(property "Dialectric" "X5R"
 			(at 230.124 111.252 0)
 			(effects
@@
 			)
 		)
-		(property "Voltage Rating" "25V"
+		(property "Voltage Rating" "16V"
 			(at 229.87 113.03 0)
 			(effects
@@
 		)
 		(property "DKN" ""
+			(at 224.79 111.76 0)
+			(effects
+				(font
+					(size 1.27 1.27)
+				)
+				(hide yes)
+			)
+		)
+		(property "JLC_PN" "C237493"
 			(at 224.79 111.76 0)
 			(effects
@@
 			)
 		)
+		(property "JLC_PN" ""
+			(at 194.31 102.87 0)
+			(effects
+				(font
+					(size 1.27 1.27)
+				)
+				(hide yes)
+			)
+		)
 		(pin "1"
 		)
@@
 			)
 		)
+		(property "JLC_PN" "C95684"
+			(at 138.43 114.3 0)
+			(effects
+				(font
+					(size 1.27 1.27)
+				)
+				(hide yes)
+			)
+		)
 		(pin "2"
 		)
@@
 		)
 		(property "DKN" ""
+			(at 204.47 102.87 0)
+			(effects
+				(font
+					(size 1.27 1.27)
+				)
+				(hide yes)
+			)
+		)
+		(property "JLC_PN" "C114626"
 			(at 204.47 102.87 0)
 			(effects
@@
 			)
 		)
-		(property "MPN" "GRM21BZ71E106KE15L"
+		(property "MPN" "GRM21BR61C106KE15K"
 			(at 88.9 95.25 0)
 			(effects
@@
 			)
 		)
-		(property "DPN" "490-GRM21BZ71E106KE15LCT-ND"
+		(property "DPN" "490-6473-1-ND"
 			(at 88.9 95.25 0)
 			(effects
@@
 			)
 		)
-		(property "Dialectric" "X7R"
+		(property "Dialectric" "X5R"
 			(at 83.566 94.742 0)
 			(effects
@@
 			)
 		)
-		(property "Voltage Rating" "25V"
+		(property "Voltage Rating" "16V"
 			(at 83.82 96.52 0)
 			(effects
@@
 		)
 		(property "DKN" ""
+			(at 88.9 95.25 0)
+			(effects
+				(font
+					(size 1.27 1.27)
+				)
+				(hide yes)
+			)
+		)
+		(property "JLC_PN" "C237493"
 			(at 88.9 95.25 0)
 			(effects
@@
 			)
 		)
-		(property "MPN" "GRM21BZ71E106KE15L"
+		(property "MPN" "GRM21BR61C106KE15K"
 			(at 165.1 95.25 0)
 			(effects
@@
 			)
 		)
-		(property "DPN" "490-GRM21BZ71E106KE15LCT-ND"
+		(property "DPN" "490-6473-1-ND"
 			(at 165.1 95.25 0)
 			(effects
@@
 			)
 		)
-		(property "Dialectric" "X7R"
+		(property "Dialectric" "X5R"
 			(at 170.434 94.742 0)
 			(effects
@@
 			)
 		)
-		(property "Voltage Rating" "25V"
+		(property "Voltage Rating" "16V"
 			(at 170.18 96.52 0)
 			(effects
@@
 		)
 		(property "DKN" ""
+			(at 165.1 95.25 0)
+			(effects
+				(font
+					(size 1.27 1.27)
+				)
+				(hide yes)
+			)
+		)
+		(property "JLC_PN" "C237493"
 			(at 165.1 95.25 0)
 			(effects
@@
 		)
 		(property "DKN" ""
+			(at 119.38 101.6 0)
+			(effects
+				(font
+					(size 1.27 1.27)
+				)
+				(hide yes)
+			)
+		)
+		(property "JLC_PN" "C25838674"
 			(at 119.38 101.6 0)
 			(effects
@@
 			)
 		)
+		(property "JLC_PN" ""
+			(at 180.34 88.9 0)
+			(effects
+				(font
+					(size 1.27 1.27)
+				)
+				(hide yes)
+			)
+		)
 		(pin "1"
 		)
@@
 			)
 		)
-		(property "MPN" "GRM21BZ71E106KE15L"
+		(property "MPN" "GRM21BR61C106KE15K"
 			(at 212.09 111.76 0)
 			(effects
@@
 			)
 		)
-		(property "DPN" "490-GRM21BZ71E106KE15LCT-ND"
+		(property "DPN" "490-6473-1-ND"
 			(at 212.09 111.76 0)
 			(effects
@@
 			)
 		)
-		(property "Dialectric" "X7R"
+		(property "Dialectric" "X5R"
 			(at 217.424 111.252 0)
 			(effects
@@
 			)
 		)
-		(property "Voltage Rating" "25V"
+		(property "Voltage Rating" "16V"
 			(at 217.17 113.03 0)
 			(effects
@@
 		)
 		(property "DKN" ""
+			(at 212.09 111.76 0)
+			(effects
+				(font
+					(size 1.27 1.27)
+				)
+				(hide yes)
+			)
+		)
+		(property "JLC_PN" "C237493"
 			(at 212.09 111.76 0)
 			(effects
@@
 			)
 		)
-		(property "Footprint" "Inductor_SMD:L_Murata_DFE201610P"
+		(property "Footprint" "ap_built:L_Murata_DFE201610P"
 			(at 143.51 88.9 0)
 			(effects
@@
 			(at 143.51 88.9 0)
 			(effects
+				(font
+					(size 1.27 1.27)
+				)
+				(hide yes)
+			)
+		)
+		(property "JLC_PN" "C882953"
+			(at 143.51 88.9 0)
+			(effects
