File: KSS_V50_HW/MCU_Prog_Comm.kicad_sch (KiCad schematic)
At the start: 16 parts, among them J5 Conn_01x04_Pin, J6 Conn_01x04_Pin, U12 SN74AUP1T34DCK, U13 SN74AUP1T34DCK, U14 SN74AUP1T34DCK, U15 SN74AUP1T34DCK

Commit message: post assembly commit
Parts:
- removed J5, J6: Conn_01x04_Pin, ap_built:Debug_Header, symbol Connector:Conn_01x04_Pin
- added J5: Conn_01x07_Pin, Connector_PinHeader_2.54mm:PinHeader_1x07_P2.54mm_Horizontal, symbol Connector:Conn_01x07_Pin
- C34, C35, C36, C37, C38, C39, C40, C41: JLC_PN (none) -> C92490
- D1: JLC_PN (none) -> C99683
- R38: JLC_PN (none) -> C144657
- U12, U13, U14, U15: JLC_PN (none) -> C131985
Connections:
- net +V_COMM_EXT is gone; now on net +V_PROG_EXT: C38.1, C40.1, U14.5 (VCCB), U15.1 (VCCA)
- net +V_PROG_EXT: now also J5.1 (Pin_1)
- net GND: now also J5.6 (Pin_6)
- net RX_COMM_EXT: now also J5.4 (Pin_4)
- net RX_PROG_EXT: now also J5.2 (Pin_2)
- net TX_COMM_EXT: now also J5.5 (Pin_5)
- net TX_PROG_EXT: now also J5.3 (Pin_3)
- new net +V_BAT: J5.7 (Pin_7)
