File: KSS_V50_HW/Motor_Driver.kicad_sch (KiCad schematic)
At the start: 19 parts, among them J3 Conn_01x04_Socket, U6 TMAG5328, U7 TMC2300-LA-T

Commit message: post assembly commit
Parts:
- added J7: Conn_01x04_Socket, Connector_Molex:Molex_PicoBlade_53261-0471_1x04-1MP_P1.25mm_Horizontal, symbol Connector:Conn_01x04_Socket
- C18, C19, C21, C22: JLC_PN (none) -> C92490
- C20: DPN 490-GRM21BZ71E106KE15LCT-ND -> 490-6473-1-ND; Dialectric X7R -> X5R; JLC_PN (none) -> C237493; MPN GRM21BZ71E106KE15L -> GRM21BR61C106KE15K; Voltage Rating 25V -> 16V
- R18, R41, R43, R45: JLC_PN (none) -> C116677
- R19, R20: JLC_PN (none) -> C114626
- R21, R22, R23: JLC_PN (none) -> C105578
- U6: JLC_PN (none) -> C5220641
- U7: footprint Package_DFN_QFN:QFN-20-1EP_3x3mm_P0.4mm_EP1.65x1.65mm -> ap_built:QFN-20-1EP_3x3mm_P0.4mm_EP1.65x1.65mm; DPN (none) -> 175-TMC2300-LA-TCT-ND; JLC_PN (none) -> C516356; MPN (none) -> TMC2300-LA-T
- renumbered J3 to J2
Connections:
- net OA1: now also J7.1 (Pin_1)
- net OA2: now also J7.2 (Pin_2)
- net OB1: now also J7.3 (Pin_3)
- net OB2: now also J7.4 (Pin_4)
Other:
- moved on the sheet: J2
